Commit message: rename package

File: techtrix_urdf_factory/urdf/bin/bin.urdf.xacro (robot description, xacro)
@@ -7,5 +7,5 @@
         <origin xyz="0 0 0" rpy="0 0 0" />
         <geometry>
-          <mesh filename="package://techtrix_gazebo/meshes/bin/visual/bin.dae" />
+          <mesh filename="package://techtrix_urdf_factory/meshes/bin/visual/bin.dae" />
         </geometry>
       </visual>
@@ -13,5 +13,5 @@
         <origin xyz="0 0 0" rpy="0 0 0"/>
         <geometry>
-          <mesh filename="package://techtrix_gazebo/meshes/bin/collision/bin_bottom.dae"/>
+          <mesh filename="package://techtrix_urdf_factory/meshes/bin/collision/bin_bottom.dae"/>
         </geometry>
       </collision>
@@ -19,12 +19,10 @@
         <origin xyz="0 0 0" rpy="0 0 0"/>
         <geometry>
-          <mesh filename="package://techtrix_gazebo/meshes/bin/collision/bin_sides.dae"/>
+          <mesh filename="package://techtrix_urdf_factory/meshes/bin/collision/bin_sides.dae"/>
         </geometry>
       </collision>
       <inertial>
         <origin xyz="0 0 0" rpy="0 0 0" />
-        <inertia ixx="1.0" ixy="0" ixz="0"
-                 iyy="1.0" iyz="0"
-                 izz="1.0" />
+        <inertia ixx="1.0" ixy="0" ixz="0" iyy="1.0" iyz="0" izz="1.0" />
         <mass value="100" />
       </inertial>
@@ -33,7 +31,5 @@
       <inertial>
         <origin xyz="0 0 0" rpy="0 0 0" />
-        <inertia ixx="1.0" ixy="0" ixz="0"
-                 iyy="1.0" iyz="0"
-                 izz="1.0" />
+        <inertia ixx="1.0" ixy="0" ixz="0" iyy="1.0" iyz="0" izz="1.0" />
         <mass value="1.0" />
       </inertial>

File: techtrix_urdf_factory/urdf/bin/bin.xacro (robot description, xacro)
@@ -1,10 +1,11 @@
 <?xml version="1.0"?>
-<robot name="bin" xmlns:xacro="http://www.ros.org/wiki/xacro">
+<robot name="bin"
+  xmlns:xacro="http://www.ros.org/wiki/xacro">
   <xacro:arg name="prefix" default="bin_1_"/>
   <!-- URDF -->
-  <xacro:include filename="$(find techtrix_gazebo)/urdf/bin/bin.urdf.xacro"/>
+  <xacro:include filename="$(find techtrix_urdf_factory)/urdf/bin/bin.urdf.xacro"/>
   <xacro:bin_urdf prefix="$(arg prefix)"/>
   <!-- Gazebo -->
-  <xacro:include filename="$(find techtrix_gazebo)/urdf/bin/bin.gazebo.xacro"/>
+  <xacro:include filename="$(find techtrix_urdf_factory)/urdf/bin/bin.gazebo.xacro"/>
   <xacro:bin_gazebo prefix="$(arg prefix)"/>
 </robot>

File: techtrix_urdf_factory/urdf/hrwros.xacro (robot description, xacro)
@@ -1,22 +1,23 @@
 <?xml version="1.0" ?>
-<robot name="robot" xmlns:xacro="http://www.ros.org/wiki/xacro">
+<robot name="robot"
+  xmlns:xacro="http://www.ros.org/wiki/xacro">
   <!-- world -->
   <link name="world" />
   <!-- workcell -->
-  <xacro:include filename="$(find techtrix_gazebo)/urdf/workcell/workcell.urdf.xacro"/>
+  <xacro:include filename="$(find techtrix_urdf_factory)/urdf/workcell/workcell.urdf.xacro"/>
   <xacro:workcell_urdf workcell_parent="world_interface"/>
   <!-- Robot1 Pedestal -->
-  <xacro:include filename="$(find techtrix_gazebo)/urdf/robot_pedestal/robot_pedestal.urdf.xacro"/>
+  <xacro:include filename="$(find techtrix_urdf_factory)/urdf/robot_pedestal/robot_pedestal.urdf.xacro"/>
   <xacro:robot_pedestal_urdf pedestal_prefix="robot1_" pedestal_parent="world_interface" pedestal_height="0.95">
     <origin xyz="0.5 1.8 0.0" rpy="0 0 0"/>
   </xacro:robot_pedestal_urdf>
   <!-- Robot1 -->
-  <xacro:include filename="$(find techtrix_gazebo)/urdf/robot_model/ur10.urdf.xacro"/>
+  <xacro:include filename="$(find techtrix_urdf_factory)/urdf/robot_model/ur10.urdf.xacro"/>
   <xacro:ur10_robot prefix="robot1_" joint_limited="true"/>
   <!-- Vacuum Gripper1 -->
-  <xacro:include filename="$(find techtrix_gazebo)/urdf/vacuum_gripper/vacuum_gripper.urdf.xacro"/>
+  <xacro:include filename="$(find techtrix_urdf_factory)/urdf/vacuum_gripper/vacuum_gripper.urdf.xacro"/>
   <xacro:vacuum_gripper_urdf prefix="vacuum_gripper1_" joint_prefix="vacuum_gripper1_joint"/>
   <!-- bins -->
-  <!-- <xacro:include filename="$(find techtrix_gazebo)/urdf/bin/bin.urdf.xacro"/>
+  <!-- <xacro:include filename="$(find techtrix_urdf_factory)/urdf/bin/bin.urdf.xacro"/>
   <xacro:bin_urdf prefix="bin_1_"/>
   <xacro:bin_urdf prefix="bin_2_"/>
@@ -37,7 +38,7 @@
   <!-- robot1 to pedestal. -->
   <joint name="robot1_to_pedestal" type="fixed">
-  <origin xyz="0 0 0.95" rpy="0 0 0" />
-  <parent link="robot1_pedestal_link" />
-  <child link="robot1_base_link" />
+    <origin xyz="0 0 0.95" rpy="0 0 0" />
+    <parent link="robot1_pedestal_link" />
+    <child link="robot1_base_link" />
   </joint>
   <!-- gripper1 to robot1. -->

File: techtrix_urdf_factory/urdf/robot_model/ur10.urdf.xacro (robot description, xacro)
@@ -1,31 +1,21 @@
 <?xml version="1.0"?>
 <robot xmlns:xacro="http://wiki.ros.org/xacro">
-<!--
+  <!--
   Author: Kelsey Hawkins
   Contributers: Jimmy Da Silva, Ajit Krisshna N L, Muhammad Asif Rana
 -->
-  <xacro:include filename="$(find techtrix_gazebo)/urdf/robot_model/ur.transmission.xacro" />
-  <xacro:include filename="$(find techtrix_gazebo)/urdf/robot_model/ur.gazebo.xacro" />
+  <xacro:include filename="$(find techtrix_urdf_factory)/urdf/robot_model/ur.transmission.xacro" />
+  <xacro:include filename="$(find techtrix_urdf_factory)/urdf/robot_model/ur.gazebo.xacro" />
   <xacro:macro name="cylinder_inertial" params="radius length mass *origin">
     <inertial>
       <mass value="${mass}" />
       <xacro:insert_block name="origin" />
-      <inertia ixx="${0.0833333 * mass * (3 * radius * radius + length * length)}" ixy="0.0" ixz="0.0"
-        iyy="${0.0833333 * mass * (3 * radius * radius + length * length)}" iyz="0.0"
-        izz="${0.5 * mass * radius * radius}" />
+      <inertia ixx="${0.0833333 * mass * (3 * radius * radius + length * length)}" ixy="0.0" ixz="0.0" iyy="${0.0833333 * mass * (3 * radius * radius + length * length)}" iyz="0.0" izz="${0.5 * mass * radius * radius}" />
     </inertial>
   </xacro:macro>
-  <xacro:macro name="ur10_robot" params="prefix joint_limited
-    shoulder_pan_lower_limit:=${-pi}    shoulder_pan_upper_limit:=${pi}
-    shoulder_lift_lower_limit:=${-pi}    shoulder_lift_upper_limit:=${pi}
-    elbow_joint_lower_limit:=${-pi}    elbow_joint_upper_limit:=${pi}
-    wrist_1_lower_limit:=${-pi}    wrist_1_upper_limit:=${pi}
-    wrist_2_lower_limit:=${-pi}    wrist_2_upper_limit:=${pi}
-    wrist_3_lower_limit:=${-pi}    wrist_3_upper_limit:=${pi}
-    transmission_hw_interface:=hardware_interface/PositionJointInterface
-    safety_limits:=false safety_pos_margin:=0.15
-    safety_k_position:=20">
+  <xacro:macro name="ur10_robot" params="prefix joint_limited shoulder_pan_lower_limit:=${-pi} shoulder_pan_upper_limit:=${pi} shoulder_lift_lower_limit:=${-pi} shoulder_lift_upper_limit:=${pi} elbow_joint_lower_limit:=${-pi} elbow_joint_upper_limit:=${pi} wrist_1_lower_limit:=${-pi} wrist_1_upper_limit:=${pi} wrist_2_lower_limit:=${-pi} wrist_2_upper_limit:=${pi} wrist_3_lower_limit:=${-pi} wrist_3_upper_limit:=${pi} transmission_hw_interface:=hardware_interface/PositionJointInterface safety_limits:=false safety_pos_margin:=0.15 safety_k_position:=20">
     <!-- Inertia parameters -->
-    <xacro:property name="base_mass" value="4.0" />  <!-- This mass might be incorrect -->
+    <xacro:property name="base_mass" value="4.0" />
+    <!-- This mass might be incorrect -->
     <xacro:property name="shoulder_mass" value="7.778" />
     <xacro:property name="upper_arm_mass" value="12.93" />
@@ -53,7 +43,10 @@
     <xacro:property name="d6" value="0.0922" />
     <!-- Arbitrary offsets for shoulder/elbow joints -->
-    <xacro:property name="shoulder_offset" value="0.220941" />  <!-- measured from model -->
-    <xacro:property name="elbow_offset" value="-0.1719" /> <!-- measured from model -->
-    <xacro:property name="upper_arm_inertia_offset" value="0.045" />  <!-- measured from model -->
+    <xacro:property name="shoulder_offset" value="0.220941" />
+    <!-- measured from model -->
+    <xacro:property name="elbow_offset" value="-0.1719" />
+    <!-- measured from model -->
+    <xacro:property name="upper_arm_inertia_offset" value="0.045" />
+    <!-- measured from model -->
     <!-- link lengths used in model -->
     <xacro:property name="shoulder_height" value="${d1}" />
@@ -63,16 +56,16 @@
     <xacro:property name="wrist_2_length" value="${d5}" />
     <xacro:property name="wrist_3_length" value="${d6}" />
-    <link name="${prefix}base_link" >
-      <visual>
-        <geometry>
-          <mesh filename="package://techtrix_gazebo/urdf/robot_model/meshes/visual/base.dae"/>
-        </geometry>
-        <material name="LightGrey">
-          <color rgba="0.7 0.7 0.7 1.0"/>
-        </material>
-      </visual>
-      <collision>
-        <geometry>
-          <mesh filename="package://techtrix_gazebo/urdf/robot_model/meshes/collision/base.stl"/>
+    <link name="${prefix}base_link">
+      <visual>
+        <geometry>
+          <mesh filename="package://techtrix_urdf_factory/urdf/robot_model/meshes/visual/base.dae"/>
+        </geometry>
+        <material name="LightGrey">
+          <color rgba="0.7 0.7 0.7 1.0"/>
+        </material>
+      </visual>
+      <collision>
+        <geometry>
+          <mesh filename="package://techtrix_urdf_factory/urdf/robot_model/meshes/collision/base.stl"/>
         </geometry>
       </collision>
@@ -103,13 +96,13 @@
       <visual>
         <geometry>
-          <mesh filename="package://techtrix_gazebo/urdf/robot_model/meshes/visual/shoulder.dae"/>
-        </geometry>
-        <material name="LightGrey">
-          <color rgba="0.7 0.7 0.7 1.0"/>
-        </material>
-      </visual>
-      <collision>
-        <geometry>
-          <mesh filename="package://techtrix_gazebo/urdf/robot_model/meshes/collision/shoulder.stl"/>
+          <mesh filename="package://techtrix_urdf_factory/urdf/robot_model/meshes/visual/shoulder.dae"/>
+        </geometry>
+        <material name="LightGrey">
+          <color rgba="0.7 0.7 0.7 1.0"/>
+        </material>
+      </visual>
+      <collision>
+        <geometry>
+          <mesh filename="package://techtrix_urdf_factory/urdf/robot_model/meshes/collision/shoulder.stl"/>
         </geometry>
       </collision>
@@ -140,13 +133,13 @@
       <visual>
         <geometry>
-          <mesh filename="package://techtrix_gazebo/urdf/robot_model/meshes/visual/upperarm.dae"/>
-        </geometry>
-        <material name="LightGrey">
-          <color rgba="0.7 0.7 0.7 1.0"/>
-        </material>
-      </visual>
-      <collision>
-        <geometry>
-          <mesh filename="package://techtrix_gazebo/urdf/robot_model/meshes/collision/upperarm.stl"/>
+          <mesh filename="package://techtrix_urdf_factory/urdf/robot_model/meshes/visual/upperarm.dae"/>
+        </geometry>
+        <material name="LightGrey">
+          <color rgba="0.7 0.7 0.7 1.0"/>
+        </material>
+      </visual>
+      <collision>
+        <geometry>
+          <mesh filename="package://techtrix_urdf_factory/urdf/robot_model/meshes/collision/upperarm.stl"/>
         </geometry>
       </collision>
@@ -176,14 +169,14 @@
     <link name="${prefix}forearm_link">
       <visual>
-         <geometry>
-          <mesh filename="package://techtrix_gazebo/urdf/robot_model/meshes/visual/forearm.dae"/>
-        </geometry>
-        <material name="LightGrey">
-          <color rgba="0.7 0.7 0.7 1.0"/>
-        </material>
-      </visual>
-      <collision>
-        <geometry>
-          <mesh filename="package://techtrix_gazebo/urdf/robot_model/meshes/collision/forearm.stl"/>
+        <geometry>
+          <mesh filename="package://techtrix_urdf_factory/urdf/robot_model/meshes/visual/forearm.dae"/>
+        </geometry>
+        <material name="LightGrey">
+          <color rgba="0.7 0.7 0.7 1.0"/>
+        </material>
+      </visual>
+      <collision>
+        <geometry>
+          <mesh filename="package://techtrix_urdf_factory/urdf/robot_model/meshes/collision/forearm.stl"/>
         </geometry>
       </collision>
@@ -214,13 +207,13 @@
       <visual>
         <geometry>
-          <mesh filename="package://techtrix_gazebo/urdf/robot_model/meshes/visual/wrist1.dae"/>
-        </geometry>
-        <material name="LightGrey">
-          <color rgba="0.7 0.7 0.7 1.0"/>
-        </material>
-      </visual>
-      <collision>
-        <geometry>
-          <mesh filename="package://techtrix_gazebo/urdf/robot_model/meshes/collision/wrist1.stl"/>
+          <mesh filename="package://techtrix_urdf_factory/urdf/robot_model/meshes/visual/wrist1.dae"/>
+        </geometry>
+        <material name="LightGrey">
+          <color rgba="0.7 0.7 0.7 1.0"/>
+        </material>
+      </visual>
+      <collision>
+        <geometry>
+          <mesh filename="package://techtrix_urdf_factory/urdf/robot_model/meshes/collision/wrist1.stl"/>
         </geometry>
       </collision>
@@ -251,13 +244,13 @@
       <visual>
         <geometry>
-          <mesh filename="package://techtrix_gazebo/urdf/robot_model/meshes/visual/wrist2.dae"/>
-        </geometry>
-        <material name="LightGrey">
-          <color rgba="0.7 0.7 0.7 1.0"/>
-        </material>
-      </visual>
-      <collision>
-        <geometry>
-          <mesh filename="package://techtrix_gazebo/urdf/robot_model/meshes/collision/wrist2.stl"/>
+          <mesh filename="package://techtrix_urdf_factory/urdf/robot_model/meshes/visual/wrist2.dae"/>
+        </geometry>
+        <material name="LightGrey">
+          <color rgba="0.7 0.7 0.7 1.0"/>
+        </material>
+      </visual>
+      <collision>
+        <geometry>
+          <mesh filename="package://techtrix_urdf_factory/urdf/robot_model/meshes/collision/wrist2.stl"/>
         </geometry>
       </collision>
@@ -288,13 +281,13 @@
       <visual>
         <geometry>
-          <mesh filename="package://techtrix_gazebo/urdf/robot_model/meshes/visual/wrist3.dae"/>
-        </geometry>
-        <material name="LightGrey">
-          <color rgba="0.7 0.7 0.7 1.0"/>
-        </material>
-      </visual>
-      <collision>
-        <geometry>
-          <mesh filename="package://techtrix_gazebo/urdf/robot_model/meshes/collision/wrist3.stl"/>
+          <mesh filename="package://techtrix_urdf_factory/urdf/robot_model/meshes/visual/wrist3.dae"/>
+        </geometry>
+        <material name="LightGrey">
+          <color rgba="0.7 0.7 0.7 1.0"/>
+        </material>
+      </visual>
+      <collision>
+        <geometry>
+          <mesh filename="package://techtrix_urdf_factory/urdf/robot_model/meshes/collision/wrist3.stl"/>
         </geometry>
       </collision>

File: techtrix_urdf_factory/urdf/robot_pedestal/robot1_pedestal.xacro (robot description, xacro)
@@ -1,4 +1,5 @@
 <?xml version="1.0" ?>
-<robot name="robot_pedestal" xmlns:xacro="http://www.ros.org/wiki/xacro">
+<robot name="robot_pedestal"
+  xmlns:xacro="http://www.ros.org/wiki/xacro">
   <xacro:arg name="pedestal_prefix" default="robot1"/>
   <xacro:arg name="pedestal_parent" default="world_interface"/>
@@ -6,9 +7,9 @@
   <link name="world_interface"/>
   <!-- URDF -->
-  <xacro:include filename="$(find techtrix_gazebo)/urdf/robot_pedestal/robot_pedestal.urdf.xacro"/>
+  <xacro:include filename="$(find techtrix_urdf_factory)/urdf/robot_pedestal/robot_pedestal.urdf.xacro"/>
   <xacro:robot_pedestal_urdf pedestal_prefix="$(arg pedestal_prefix)" pedestal_parent="$(arg pedestal_parent)" pedestal_height="$(arg pedestal_height)">
     <origin xyz="0.5 1.8 0.0" rpy="0 0 0"/>
   </xacro:robot_pedestal_urdf>
   <!-- Gazebo -->
-  <xacro:include filename="$(find techtrix_gazebo)/urdf/robot_pedestal/robot_pedestal.gazebo.xacro"/>
+  <xacro:include filename="$(find techtrix_urdf_factory)/urdf/robot_pedestal/robot_pedestal.gazebo.xacro"/>
 </robot>

File: techtrix_urdf_factory/urdf/robot_pedestal/robot2_pedestal.xacro (robot description, xacro)
@@ -1,4 +1,5 @@
 <?xml version="1.0" ?>
-<robot name="robot2_pedestal" xmlns:xacro="http://www.ros.org/wiki/xacro">
+<robot name="robot2_pedestal"
+  xmlns:xacro="http://www.ros.org/wiki/xacro">
   <xacro:arg name="pedestal_prefix" default="robot1"/>
   <xacro:arg name="pedestal_parent" default="world_interface"/>
@@ -6,9 +7,9 @@
   <link name="world_interface"/>
   <!-- URDF -->
-  <xacro:include filename="$(find techtrix_gazebo)/urdf/robot_pedestal/robot_pedestal.urdf.xacro"/>
+  <xacro:include filename="$(find techtrix_urdf_factory)/urdf/robot_pedestal/robot_pedestal.urdf.xacro"/>
   <xacro:robot_pedestal_urdf pedestal_prefix="$(arg pedestal_prefix)" pedestal_parent="$(arg pedestal_parent)" pedestal_height="$(arg pedestal_height)">
     <origin xyz="-7.8 -1.5 0.0" rpy="0 0 0"/>
   </xacro:robot_pedestal_urdf>
   <!-- Gazebo -->
-  <xacro:include filename="$(find techtrix_gazebo)/urdf/robot_pedestal/robot_pedestal.gazebo.xacro"/>
+  <xacro:include filename="$(find techtrix_urdf_factory)/urdf/robot_pedestal/robot_pedestal.gazebo.xacro"/>
 </robot>

File: techtrix_urdf_factory/urdf/vacuum_gripper/vacuum_gripper.urdf.xacro (robot description, xacro)
@@ -7,5 +7,5 @@
         <origin xyz="0 0 0" rpy="0 0 0" />
         <geometry>
-          <mesh filename="package://techtrix_gazebo/meshes/vacuum_gripper/visual/vacuum_gripper.dae"/>
+          <mesh filename="package://techtrix_urdf_factory/meshes/vacuum_gripper/visual/vacuum_gripper.dae"/>
         </geometry>
         <material name="red">
@@ -16,5 +16,5 @@
         <origin xyz="0 0 0" rpy="0 0 0"/>
         <geometry>
-          <mesh filename="package://techtrix_gazebo/meshes/vacuum_gripper/collision/vacuum_gripper.dae"/>
+          <mesh filename="package://techtrix_urdf_factory/meshes/vacuum_gripper/collision/vacuum_gripper.dae"/>
         </geometry>
         <material name="red"/>
@@ -22,7 +22,5 @@
       <inertial>
         <origin xyz="0 0 0" rpy="0 0 0" />
-        <inertia ixx="1.0" ixy="0" ixz="0"
-                 iyy="1.0" iyz="0"
-                 izz="1.0" />
+        <inertia ixx="1.0" ixy="0" ixz="0" iyy="1.0" iyz="0" izz="1.0" />
         <mass value="1.0" />
       </inertial>
@@ -47,7 +45,5 @@
       <inertial>
         <origin xyz="0 0 0" rpy="0 0 0" />
-        <inertia ixx="0.0001" ixy="0" ixz="0"
-                 iyy="0.0001" iyz="0"
-                 izz="0.0001" />
+        <inertia ixx="0.0001" ixy="0" ixz="0" iyy="0.0001" iyz="0" izz="0.0001" />
         <mass value="0.00001" />
       </inertial>

File: techtrix_urdf_factory/urdf/vacuum_gripper/vacuum_gripper.xacro (robot description, xacro)
@@ -1,10 +1,11 @@
 <?xml version="1.0"?>
-<robot name="vacuum_gripper" xmlns:xacro="http://www.ros.org/wiki/xacro">
+<robot name="vacuum_gripper"
+  xmlns:xacro="http://www.ros.org/wiki/xacro">
   <xacro:arg name="prefix" default="vacuum_gripper_"/>
   <!-- URDF -->
-  <xacro:include filename="$(find techtrix_gazebo)/urdf/vacuum_gripper/vacuum_gripper.urdf.xacro"/>
+  <xacro:include filename="$(find techtrix_urdf_factory)/urdf/vacuum_gripper/vacuum_gripper.urdf.xacro"/>
   <xacro:vacuum_gripper_urdf prefix="$(arg prefix)"/>
   <!-- Gazebo -->
-  <xacro:include filename="$(find techtrix_gazebo)/urdf/vacuum_gripper/vacuum_gripper.gazebo.xacro"/>
+  <xacro:include filename="$(find techtrix_urdf_factory)/urdf/vacuum_gripper/vacuum_gripper.gazebo.xacro"/>
   <xacro:vacuum_gripper_gazebo prefix="$(arg prefix)" gripper_link="${prefix}::${prefix}tool0">
     <drops_info/>

File: techtrix_urdf_factory/urdf/workcell/workcell.urdf.xacro (robot description, xacro)
@@ -1,5 +1,6 @@
 <?xml version="1.0" ?>
-<robot name="workcell_urdf" xmlns:xacro="http://www.ros.org/wiki/xacro">
-    <xacro:macro name="workcell_urdf" params="workcell_parent">
+<robot name="workcell_urdf"
+  xmlns:xacro="http://www.ros.org/wiki/xacro">
+  <xacro:macro name="workcell_urdf" params="workcell_parent">
     <!-- Links -->
     <link name="world_interface"/>
@@ -7,16 +8,14 @@
       <visual>
         <geometry>
-          <mesh filename="package://techtrix_gazebo/meshes/workcell/visual/workcell.dae"/>
+          <mesh filename="package://techtrix_urdf_factory/meshes/workcell/visual/workcell.dae"/>
         </geometry>
       </visual>
       <collision>
         <geometry>
-          <mesh filename="package://techtrix_gazebo/meshes/workcell/collision/workcell.dae"/>
+          <mesh filename="package://techtrix_urdf_factory/meshes/workcell/collision/workcell.dae"/>
         </geometry>
       </collision>
       <inertial>
-        <inertia ixx="1.0" ixy="0" ixz="0"
-                 iyy="1.0" iyz="0"
-                 izz="1.0" />
+        <inertia ixx="1.0" ixy="0" ixz="0" iyy="1.0" iyz="0" izz="1.0" />
         <mass value="100" />
       </inertial>

File: techtrix_urdf_factory/urdf/workcell/workcell.xacro (robot description, xacro)
@@ -1,9 +1,10 @@
 <?xml version="1.0" ?>
-<robot name="workcell" xmlns:xacro="http://www.ros.org/wiki/xacro">
+<robot name="workcell"
+  xmlns:xacro="http://www.ros.org/wiki/xacro">
   <xacro:arg name="workcell_parent_name" default="world_interface"/>
   <!-- URDF -->
-  <xacro:include filename="$(find techtrix_gazebo)/urdf/workcell/workcell.urdf.xacro"/>
+  <xacro:include filename="$(find techtrix_urdf_factory)/urdf/workcell/workcell.urdf.xacro"/>
   <xacro:workcell_urdf workcell_parent="$(arg workcell_parent_name)"/>
   <!-- Gazebo -->
-  <xacro:include filename="$(find techtrix_gazebo)/urdf/workcell/workcell.gazebo.xacro"/>
+  <xacro:include filename="$(find techtrix_urdf_factory)/urdf/workcell/workcell.gazebo.xacro"/>
 </robot>
