Commit message: Added Rviz support for the camera sensor

File: techtrix_description/urdf/gazebo_plugins.xacro (robot description, xacro)
@@ -2,7 +2,12 @@
 <robot xmlns:xacro="http://www.ros.org/wiki/xacro" name="techtrix_robot">
   <!-- camera -->
-  <gazebo reference="camera_link">
-    <sensor type="camera" name="camera1">
-      <update_rate>30.0</update_rate>
+  <gazebo reference="camera_link"> <!--The link name must match the link name of the URDF model -->
+    <sensor type="camera" name="camera1"> <!-- The name "camera1" must be unique from all other sensors -->
+      <update_rate>30.0</update_rate> <!-- Number of times per second a new camera image is taken within Gazebo -->
+                                      <!-- This is the maximum update rate the sensor will attempt during simulation
+                                           but it could fall behind this target rate if the physics simulation runs
+                                           faster than the sensor generation can keep up.-->
+      <!-- Next, we set upp the manufacturer;s spects of our physical camera hardware -->
+      <!-- Note that the pixels are assumed to be square -->
       <camera name="head">
         <horizontal_fov>1.3962634</horizontal_fov>
@@ -12,4 +17,8 @@
           <format>R8G8B8</format>
         </image>
+        <!-- The near and far clips are simulation-specific
+             parameters that give an upper and lower bound to the distance
+             in which the cameras can see objects in the simulation.
+             This is specified in the camera's optometry frame. -->
         <clip>
           <near>0.02</near>
@@ -25,10 +34,17 @@
         </noise>
       </camera>
+      <!-- This is where the actual gazebo_ros/gazebo_ros_camera.cpp file is linked to, as a shared object -->
       <plugin name="camera_controller" filename="libgazebo_ros_camera.so">
         <alwaysOn>true</alwaysOn>
         <updateRate>0.0</updateRate>
-        <cameraName>rrbot/camera1</cameraName>
+        <!-- We define the rostopic the camera will be publishing to, for both the image topic and the camera info topic -->
+        <cameraName>techtrix/camera1</cameraName>
         <imageTopicName>image_raw</imageTopicName>
         <cameraInfoTopicName>camera_info</cameraInfoTopicName>
+        <!-- Hence, for techtrix robot, you should subscribe to:
+             /techtrix/camera1/image_raw
+             /techtrix/camera1/camera_info-->
+        <!-- Finally, we set the coordinate frame the image
+             is published under in the tf tree.-->
         <frameName>camera_link</frameName>
         <hackBaseline>0.07</hackBaseline>

File: techtrix_description/urdf/techtrix.xacro (robot description, xacro)
@@ -52,5 +52,7 @@
 	      <box size="${camera_link} ${camera_link} ${camera_link}"/>
       </geometry>
-      <material name="red"/>
+      <material name="yellow">
+        <color rgba="1 1 0 1"/>
+      </material>
     </visual>
     <inertial>

Commit message: Add laser sensors

File: techtrix_description/urdf/gazebo_plugins.xacro (robot description, xacro)
@@ -182,3 +182,164 @@
     </sensor>
   </gazebo>
+  <gazebo reference="grabbing_mechanism_l">
+    <sensor type="ray" name="sc_1_laser">
+      <visualize>true</visualize>
+      <update_rate>40</update_rate>
+      <ray>
+        <scan>
+          <horizontal>
+            <samples>10</samples>
+            <resolution>1</resolution>
+            <min_angle>0</min_angle>
+            <max_angle>0</max_angle>
+          </horizontal>
+        </scan>
+        <range>
+          <min>0.1</min>
+          <max>30.0</max>
+          <resolution>0.01</resolution>
+        </range>
+      </ray>
+      <plugin name="sc_1_laser_controller" filename="libgazebo_ros_laser.so">
+        <robotNamespace>techtrix</robotNamespace>
+        <topicName>/techtrix/laser/sc_1</topicName>
+        <frameName>grabbing_mechanism_l</frameName>
+      </plugin>
+    </sensor>
+  </gazebo>
+  <gazebo reference="grabbing_mechanism">
+    <sensor type="ray" name="sc_2_laser">
+      <pose>0.339 0 0 0 ${pi/2} 0</pose>
+      <visualize>true</visualize>
+      <update_rate>40</update_rate>
+      <ray>
+        <scan>
+          <horizontal>
+            <samples>10</samples>
+            <resolution>1</resolution>
+            <min_angle>0</min_angle>
+            <max_angle>0</max_angle>
+          </horizontal>
+        </scan>
+        <range>
+          <min>0.0</min>
+          <max>30.0</max>
+          <resolution>0.01</resolution>
+        </range>
+      </ray>
+      <plugin name="sc_2_laser_controller" filename="libgazebo_ros_laser.so">
+        <robotNamespace>techtrix</robotNamespace>
+        <topicName>/techtrix/laser/sc_2</topicName>
+        <frameName>grabbing_mechanism</frameName>
+      </plugin>
+    </sensor>
+  </gazebo>
+  <gazebo reference="grabbing_mechanism">
+    <sensor type="ray" name="sc_3_laser">
+      <pose>0.127 0 0 0 ${pi/2} 0</pose>
+      <visualize>true</visualize>
+      <update_rate>40</update_rate>
+      <ray>
+        <scan>
+          <horizontal>
+            <samples>10</samples>
+            <resolution>1</resolution>
+            <min_angle>0</min_angle>
+            <max_angle>0</max_angle>
+          </horizontal>
+        </scan>
+        <range>
+          <min>0.0</min>
+          <max>30.0</max>
+          <resolution>0.01</resolution>
+        </range>
+      </ray>
+      <plugin name="sc_3_laser_controller" filename="libgazebo_ros_laser.so">
+        <robotNamespace>techtrix</robotNamespace>
+        <topicName>/techtrix/laser/sc_3</topicName>
+        <frameName>grabbing_mechanism</frameName>
+      </plugin>
+    </sensor>
+  </gazebo>
+  <gazebo reference="grabbing_mechanism">
+    <sensor type="ray" name="sc_4_laser">
+      <pose>-0.127 0 0 0 ${pi/2} 0</pose>
+      <visualize>true</visualize>
+      <update_rate>40</update_rate>
+      <ray>
+        <scan>
+          <horizontal>
+            <samples>10</samples>
+            <resolution>1</resolution>
+            <min_angle>0</min_angle>
+            <max_angle>0</max_angle>
+          </horizontal>
+        </scan>
+        <range>
+          <min>0.0</min>
+          <max>30.0</max>
+          <resolution>0.01</resolution>
+        </range>
+      </ray>
+      <plugin name="sc_4_laser_controller" filename="libgazebo_ros_laser.so">
+        <robotNamespace>techtrix</robotNamespace>
+        <topicName>/techtrix/laser/sc_4</topicName>
+        <frameName>grabbing_mechanism</frameName>
+      </plugin>
+    </sensor>
+  </gazebo>
+  <gazebo reference="grabbing_mechanism">
+    <sensor type="ray" name="sc_5_laser">
+      <pose>-0.339 0 0 0 ${pi/2} 0</pose>
+      <visualize>true</visualize>
+      <update_rate>40</update_rate>
+      <ray>
+        <scan>
+          <horizontal>
+            <samples>10</samples>
+            <resolution>1</resolution>
+            <min_angle>0</min_angle>
+            <max_angle>0</max_angle>
+          </horizontal>
+        </scan>
+        <range>
+          <min>0.0</min>
+          <max>30.0</max>
+          <resolution>0.01</resolution>
+        </range>
+      </ray>
+      <plugin name="sc_5_laser_controller" filename="libgazebo_ros_laser.so">
+        <robotNamespace>techtrix</robotNamespace>
+        <topicName>/techtrix/laser/sc_5</topicName>
+        <frameName>grabbing_mechanism</frameName>
+      </plugin>
+    </sensor>
+  </gazebo>
+  <gazebo reference="grabbing_mechanism">
+    <sensor type="ray" name="sc_6_laser">
+      <pose>-0.551 0 0 0 ${pi/2} 0</pose>
+      <visualize>true</visualize>
+      <update_rate>40</update_rate>
+      <ray>
+        <scan>
+          <horizontal>
+            <samples>10</samples>
+            <resolution>1</resolution>
+            <min_angle>0</min_angle>
+            <max_angle>0</max_angle>
+          </horizontal>
+        </scan>
+        <range>
+          <min>0.0</min>
+          <max>30.0</max>
+          <resolution>0.01</resolution>
+        </range>
+      </ray>
+      <plugin name="sc_6_laser_controller" filename="libgazebo_ros_laser.so">
+        <robotNamespace>techtrix</robotNamespace>
+        <topicName>/techtrix/laser/sc_6</topicName>
+        <frameName>grabbing_mechanism</frameName>
+      </plugin>
+    </sensor>
+  </gazebo>
 </robot>

File: techtrix_description/urdf/techtrix.xacro (robot description, xacro)
@@ -24,4 +24,17 @@
     <xacro:default_inertial mass="1"/>
   </link>
+    <link name="grabbing_mechanism_l">
+        <visual>
+            <origin xyz="0 0 0" rpy="0 0 0" />
+            <geometry>
+                <box size="0.1 0.1 0.1" />
+            </geometry>
+        </visual>
+    </link>
+    <joint name="cdefwamera_joint" type="fixed">
+      <origin xyz="0.551 0 0" rpy="0 0.7 0" />
+      <parent link="grabbing_mechanism"/>
+      <child link="grabbing_mechanism_l" />
+    </joint>
   <link name="grabbing_mechanism">
     <collision name="grabbing_mechanism_sc_1_top">

Commit message: Fix lasers positions and visualization

File: techtrix_description/urdf/gazebo_plugins.xacro (robot description, xacro)
@@ -182,5 +182,5 @@
     </sensor>
   </gazebo>
-  <gazebo reference="grabbing_mechanism_l">
+  <gazebo reference="grabbing_mechanism_sc_1_laser">
     <sensor type="ray" name="sc_1_laser">
       <visualize>true</visualize>
@@ -204,24 +204,23 @@
         <robotNamespace>techtrix</robotNamespace>
         <topicName>/techtrix/laser/sc_1</topicName>
-        <frameName>grabbing_mechanism_l</frameName>
-      </plugin>
-    </sensor>
-  </gazebo>
-  <gazebo reference="grabbing_mechanism">
+        <frameName>grabbing_mechanism_sc_1_laser</frameName>
+      </plugin>
+    </sensor>
+  </gazebo>
+  <gazebo reference="grabbing_mechanism_sc_2_laser">
     <sensor type="ray" name="sc_2_laser">
-      <pose>0.339 0 0 0 ${pi/2} 0</pose>
-      <visualize>true</visualize>
-      <update_rate>40</update_rate>
-      <ray>
-        <scan>
-          <horizontal>
-            <samples>10</samples>
-            <resolution>1</resolution>
-            <min_angle>0</min_angle>
-            <max_angle>0</max_angle>
-          </horizontal>
-        </scan>
-        <range>
-          <min>0.0</min>
+      <visualize>true</visualize>
+      <update_rate>40</update_rate>
+      <ray>
+        <scan>
+          <horizontal>
+            <samples>10</samples>
+            <resolution>1</resolution>
+            <min_angle>0</min_angle>
+            <max_angle>0</max_angle>
+          </horizontal>
+        </scan>
+        <range>
+          <min>0.1</min>
           <max>30.0</max>
           <resolution>0.01</resolution>
@@ -231,24 +230,23 @@
         <robotNamespace>techtrix</robotNamespace>
         <topicName>/techtrix/laser/sc_2</topicName>
-        <frameName>grabbing_mechanism</frameName>
-      </plugin>
-    </sensor>
-  </gazebo>
-  <gazebo reference="grabbing_mechanism">
+        <frameName>grabbing_mechanism_sc_2_laser</frameName>
+      </plugin>
+    </sensor>
+  </gazebo>
+  <gazebo reference="grabbing_mechanism_sc_3_laser">
     <sensor type="ray" name="sc_3_laser">
-      <pose>0.127 0 0 0 ${pi/2} 0</pose>
-      <visualize>true</visualize>
-      <update_rate>40</update_rate>
-      <ray>
-        <scan>
-          <horizontal>
-            <samples>10</samples>
-            <resolution>1</resolution>
-            <min_angle>0</min_angle>
-            <max_angle>0</max_angle>
-          </horizontal>
-        </scan>
-        <range>
-          <min>0.0</min>
+      <visualize>true</visualize>
+      <update_rate>40</update_rate>
+      <ray>
+        <scan>
+          <horizontal>
+            <samples>10</samples>
+            <resolution>1</resolution>
+            <min_angle>0</min_angle>
+            <max_angle>0</max_angle>
+          </horizontal>
+        </scan>
+        <range>
+          <min>0.1</min>
           <max>30.0</max>
           <resolution>0.01</resolution>
@@ -258,24 +256,23 @@
         <robotNamespace>techtrix</robotNamespace>
         <topicName>/techtrix/laser/sc_3</topicName>
-        <frameName>grabbing_mechanism</frameName>
-      </plugin>
-    </sensor>
-  </gazebo>
-  <gazebo reference="grabbing_mechanism">
+        <frameName>grabbing_mechanism_sc_3_laser</frameName>
+      </plugin>
+    </sensor>
+  </gazebo>
+  <gazebo reference="grabbing_mechanism_sc_4_laser">
     <sensor type="ray" name="sc_4_laser">
-      <pose>-0.127 0 0 0 ${pi/2} 0</pose>
-      <visualize>true</visualize>
-      <update_rate>40</update_rate>
-      <ray>
-        <scan>
-          <horizontal>
-            <samples>10</samples>
-            <resolution>1</resolution>
-            <min_angle>0</min_angle>
-            <max_angle>0</max_angle>
-          </horizontal>
-        </scan>
-        <range>
-          <min>0.0</min>
+      <visualize>true</visualize>
+      <update_rate>40</update_rate>
+      <ray>
+        <scan>
+          <horizontal>
+            <samples>10</samples>
+            <resolution>1</resolution>
+            <min_angle>0</min_angle>
+            <max_angle>0</max_angle>
+          </horizontal>
+        </scan>
+        <range>
+          <min>0.1</min>
           <max>30.0</max>
           <resolution>0.01</resolution>
@@ -285,24 +282,23 @@
         <robotNamespace>techtrix</robotNamespace>
         <topicName>/techtrix/laser/sc_4</topicName>
-        <frameName>grabbing_mechanism</frameName>
-      </plugin>
-    </sensor>
-  </gazebo>
-  <gazebo reference="grabbing_mechanism">
+        <frameName>grabbing_mechanism_sc_4_laser</frameName>
+      </plugin>
+    </sensor>
+  </gazebo>
+  <gazebo reference="grabbing_mechanism_sc_5_laser">
     <sensor type="ray" name="sc_5_laser">
-      <pose>-0.339 0 0 0 ${pi/2} 0</pose>
-      <visualize>true</visualize>
-      <update_rate>40</update_rate>
-      <ray>
-        <scan>
-          <horizontal>
-            <samples>10</samples>
-            <resolution>1</resolution>
-            <min_angle>0</min_angle>
-            <max_angle>0</max_angle>
-          </horizontal>
-        </scan>
-        <range>
-          <min>0.0</min>
+      <visualize>true</visualize>
+      <update_rate>40</update_rate>
+      <ray>
+        <scan>
+          <horizontal>
+            <samples>10</samples>
+            <resolution>1</resolution>
+            <min_angle>0</min_angle>
+            <max_angle>0</max_angle>
+          </horizontal>
+        </scan>
+        <range>
+          <min>0.1</min>
           <max>30.0</max>
           <resolution>0.01</resolution>
@@ -312,24 +308,23 @@
         <robotNamespace>techtrix</robotNamespace>
         <topicName>/techtrix/laser/sc_5</topicName>
-        <frameName>grabbing_mechanism</frameName>
-      </plugin>
-    </sensor>
-  </gazebo>
-  <gazebo reference="grabbing_mechanism">
+        <frameName>grabbing_mechanism_sc_5_laser</frameName>
+      </plugin>
+    </sensor>
+  </gazebo>
+  <gazebo reference="grabbing_mechanism_sc_6_laser">
     <sensor type="ray" name="sc_6_laser">
-      <pose>-0.551 0 0 0 ${pi/2} 0</pose>
-      <visualize>true</visualize>
-      <update_rate>40</update_rate>
-      <ray>
-        <scan>
-          <horizontal>
-            <samples>10</samples>
-            <resolution>1</resolution>
-            <min_angle>0</min_angle>
-            <max_angle>0</max_angle>
-          </horizontal>
-        </scan>
-        <range>
-          <min>0.0</min>
+      <visualize>true</visualize>
+      <update_rate>40</update_rate>
+      <ray>
+        <scan>
+          <horizontal>
+            <samples>10</samples>
+            <resolution>1</resolution>
+            <min_angle>0</min_angle>
+            <max_angle>0</max_angle>
+          </horizontal>
+        </scan>
+        <range>
+          <min>0.1</min>
           <max>30.0</max>
           <resolution>0.01</resolution>
@@ -339,5 +334,5 @@
         <robotNamespace>techtrix</robotNamespace>
         <topicName>/techtrix/laser/sc_6</topicName>
-        <frameName>grabbing_mechanism</frameName>
+        <frameName>grabbing_mechanism_sc_6_laser</frameName>
       </plugin>
     </sensor>

File: techtrix_description/urdf/techtrix.xacro (robot description, xacro)
@@ -24,17 +24,82 @@
     <xacro:default_inertial mass="1"/>
   </link>
-    <link name="grabbing_mechanism_l">
-        <visual>
-            <origin xyz="0 0 0" rpy="0 0 0" />
-            <geometry>
-                <box size="0.1 0.1 0.1" />
-            </geometry>
-        </visual>
-    </link>
-    <joint name="cdefwamera_joint" type="fixed">
-      <origin xyz="0.551 0 0" rpy="0 0.7 0" />
-      <parent link="grabbing_mechanism"/>
-      <child link="grabbing_mechanism_l" />
-    </joint>
+  <link name="grabbing_mechanism_sc_1_laser">
+    <visual>
+      <origin xyz="0 0 0" rpy="0 0 0" />
+      <geometry>
+        <box size="0.01 0.01 0.01" />
+      </geometry>
+    </visual>
+  </link>
+  <joint name="grabbing_mechanism_sc_1_laser_joint" type="fixed">
+    <origin xyz="0.551 0 0" rpy="0 ${pi/2} 0" />
+    <parent link="grabbing_mechanism"/>
+    <child link="grabbing_mechanism_sc_1_laser" />
+  </joint>
+  <link name="grabbing_mechanism_sc_2_laser">
+    <visual>
+      <origin xyz="0 0 0" rpy="0 0 0" />
+      <geometry>
+        <box size="0.01 0.01 0.01" />
+      </geometry>
+    </visual>
+  </link>
+  <joint name="grabbing_mechanism_sc_2_laser_joint" type="fixed">
+    <origin xyz="0.339 0 0" rpy="0 ${pi/2} 0" />
+    <parent link="grabbing_mechanism"/>
+    <child link="grabbing_mechanism_sc_2_laser" />
+  </joint>
+  <link name="grabbing_mechanism_sc_3_laser">
+    <visual>
+      <origin xyz="0 0 0" rpy="0 0 0" />
+      <geometry>
+        <box size="0.01 0.01 0.01" />
+      </geometry>
+    </visual>
+  </link>
+  <joint name="grabbing_mechanism_sc_3_laser_joint" type="fixed">
+    <origin xyz="0.127 0 0" rpy="0 ${pi/2} 0" />
+    <parent link="grabbing_mechanism"/>
+    <child link="grabbing_mechanism_sc_3_laser" />
+  </joint>
+  <link name="grabbing_mechanism_sc_4_laser">
+    <visual>
+      <origin xyz="0 0 0" rpy="0 0 0" />
+      <geometry>
+        <box size="0.01 0.01 0.01" />
+      </geometry>
+    </visual>
+  </link>
+  <joint name="grabbing_mechanism_sc_4_laser_joint" type="fixed">
+    <origin xyz="-0.127 0 0" rpy="0 ${pi/2} 0" />
+    <parent link="grabbing_mechanism"/>
+    <child link="grabbing_mechanism_sc_4_laser" />
+  </joint>
+  <link name="grabbing_mechanism_sc_5_laser">
+    <visual>
+      <origin xyz="0 0 0" rpy="0 0 0" />
+      <geometry>
+        <box size="0.01 0.01 0.01" />
+      </geometry>
+    </visual>
+  </link>
+  <joint name="grabbing_mechanism_sc_5_laser_joint" type="fixed">
+    <origin xyz="-0.339 0 0" rpy="0 ${pi/2} 0" />
+    <parent link="grabbing_mechanism"/>
+    <child link="grabbing_mechanism_sc_5_laser" />
+  </joint>
+  <link name="grabbing_mechanism_sc_6_laser">
+    <visual>
+      <origin xyz="0 0 0" rpy="0 0 0" />
+      <geometry>
+        <box size="0.01 0.01 0.01" />
+      </geometry>
+    </visual>
+  </link>
+  <joint name="grabbing_mechanism_sc_6_laser_joint" type="fixed">
+    <origin xyz="-0.551 0 0" rpy="0 ${pi/2} 0" />
+    <parent link="grabbing_mechanism"/>
+    <child link="grabbing_mechanism_sc_6_laser" />
+  </joint>
   <link name="grabbing_mechanism">
     <collision name="grabbing_mechanism_sc_1_top">
