Commit message: Fix contact sensors collisions and laser min distance

File: techtrix_description/urdf/gazebo_plugins.xacro (robot description, xacro)
@@ -13,14 +13,13 @@
         <collision_y>-0.098</collision_y>
         <collision_z>-0.135</collision_z>
-        <marker_namespace>sc_1_top</marker_namespace>
-      </plugin>
-    </sensor>
-  </gazebo>
-  <gazebo reference="grabbing_mechanism">
+        <marker_publish>sc_1_top</marker_publish>
+        <marker_id>1</marker_id>
+      </plugin>
+    </sensor>
     <sensor name='grabber_contact_sensor_sc_1_bot' type='contact'>
       <always_on>true</always_on>
       <update_rate>100</update_rate>
       <contact>
-        <collision>grabbing_mechanism_sc_1_bot_collision</collision>
+        <collision>grabbing_mechanism_sc_1_bot_collision_1</collision>
       </contact>
       <plugin name="contact_plugin_sc_1_bot" filename="libGrabberContactPlugin.so">
@@ -28,14 +27,13 @@
         <collision_y>-0.098</collision_y>
         <collision_z>-0.255</collision_z>
-        <marker_namespace>sc_1_bot</marker_namespace>
-      </plugin>
-    </sensor>
-  </gazebo>
-  <gazebo reference="grabbing_mechanism">
+        <marker_publish>sc_1_bot</marker_publish>
+        <marker_id>2</marker_id>
+      </plugin>
+    </sensor>
     <sensor name='grabber_contact_sensor_sc_2_top' type='contact'>
       <always_on>true</always_on>
       <update_rate>100</update_rate>
       <contact>
-        <collision>grabbing_mechanism_sc_2_top_collision</collision>
+        <collision>grabbing_mechanism_sc_2_top_collision_2</collision>
       </contact>
       <plugin name="contact_plugin_sc_2_top" filename="libGrabberContactPlugin.so">
@@ -43,14 +41,13 @@
         <collision_y>-0.098</collision_y>
         <collision_z>-0.135</collision_z>
-        <marker_namespace>sc_2_top</marker_namespace>
-      </plugin>
-    </sensor>
-  </gazebo>
-  <gazebo reference="grabbing_mechanism">
+        <marker_publish>sc_2_top</marker_publish>
+        <marker_id>3</marker_id>
+      </plugin>
+    </sensor>
     <sensor name='grabber_contact_sensor_sc_2_bot' type='contact'>
       <always_on>true</always_on>
       <update_rate>100</update_rate>
       <contact>
-        <collision>grabbing_mechanism_sc_2_bot_collision</collision>
+        <collision>grabbing_mechanism_sc_2_bot_collision_3</collision>
       </contact>
       <plugin name="contact_plugin_sc_2_bot" filename="libGrabberContactPlugin.so">
@@ -58,14 +55,13 @@
         <collision_y>-0.098</collision_y>
         <collision_z>-0.255</collision_z>
-        <marker_namespace>sc_2_bot</marker_namespace>
-      </plugin>
-    </sensor>
-  </gazebo>
-  <gazebo reference="grabbing_mechanism">
+        <marker_publish>sc_2_bot</marker_publish>
+        <marker_id>4</marker_id>
+      </plugin>
+    </sensor>
     <sensor name='grabber_contact_sensor_sc_3_top' type='contact'>
       <always_on>true</always_on>
       <update_rate>100</update_rate>
       <contact>
-        <collision>grabbing_mechanism_sc_3_top_collision</collision>
+        <collision>grabbing_mechanism_sc_3_top_collision_4</collision>
       </contact>
       <plugin name="contact_plugin_sc_3_top" filename="libGrabberContactPlugin.so">
@@ -73,14 +69,13 @@
         <collision_y>-0.098</collision_y>
         <collision_z>-0.135</collision_z>
-        <marker_namespace>sc_3_top</marker_namespace>
-      </plugin>
-    </sensor>
-  </gazebo>
-  <gazebo reference="grabbing_mechanism">
+        <marker_publish>sc_3_top</marker_publish>
+        <marker_id>5</marker_id>
+      </plugin>
+    </sensor>
     <sensor name='grabber_contact_sensor_sc_3_bot' type='contact'>
       <always_on>true</always_on>
       <update_rate>100</update_rate>
       <contact>
-        <collision>grabbing_mechanism_sc_3_bot_collision</collision>
+        <collision>grabbing_mechanism_sc_3_bot_collision_5</collision>
       </contact>
       <plugin name="contact_plugin_sc_3_bot" filename="libGrabberContactPlugin.so">
@@ -88,14 +83,13 @@
         <collision_y>-0.098</collision_y>
         <collision_z>-0.255</collision_z>
-        <marker_namespace>sc_3_bot</marker_namespace>
-      </plugin>
-    </sensor>
-  </gazebo>
-  <gazebo reference="grabbing_mechanism">
+        <marker_publish>sc_3_bot</marker_publish>
+        <marker_id>6</marker_id>
+      </plugin>
+    </sensor>
     <sensor name='grabber_contact_sensor_sc_4_top' type='contact'>
       <always_on>true</always_on>
       <update_rate>100</update_rate>
       <contact>
-        <collision>grabbing_mechanism_sc_4_top_collision</collision>
+        <collision>grabbing_mechanism_sc_4_top_collision_6</collision>
       </contact>
       <plugin name="contact_plugin_sc_4_top" filename="libGrabberContactPlugin.so">
@@ -103,14 +97,13 @@
         <collision_y>-0.098</collision_y>
         <collision_z>-0.135</collision_z>
-        <marker_namespace>sc_4_top</marker_namespace>
-      </plugin>
-    </sensor>
-  </gazebo>
-  <gazebo reference="grabbing_mechanism">
+        <marker_publish>sc_4_top</marker_publish>
+        <marker_id>7</marker_id>
+      </plugin>
+    </sensor>
     <sensor name='grabber_contact_sensor_sc_4_bot' type='contact'>
       <always_on>true</always_on>
       <update_rate>100</update_rate>
       <contact>
-        <collision>grabbing_mechanism_sc_4_bot_collision</collision>
+        <collision>grabbing_mechanism_sc_4_bot_collision_7</collision>
       </contact>
       <plugin name="contact_plugin_sc_4_bot" filename="libGrabberContactPlugin.so">
@@ -118,14 +111,13 @@
         <collision_y>-0.098</collision_y>
         <collision_z>-0.255</collision_z>
-        <marker_namespace>sc_4_bot</marker_namespace>
-      </plugin>
-    </sensor>
-  </gazebo>
-  <gazebo reference="grabbing_mechanism">
+        <marker_publish>sc_4_bot</marker_publish>
+        <marker_id>8</marker_id>
+      </plugin>
+    </sensor>
     <sensor name='grabber_contact_sensor_sc_5_top' type='contact'>
       <always_on>true</always_on>
       <update_rate>100</update_rate>
       <contact>
-        <collision>grabbing_mechanism_sc_5_top_collision</collision>
+        <collision>grabbing_mechanism_sc_5_top_collision_8</collision>
       </contact>
       <plugin name="contact_plugin_sc_5_top" filename="libGrabberContactPlugin.so">
@@ -133,14 +125,13 @@
         <collision_y>-0.098</collision_y>
         <collision_z>-0.135</collision_z>
-        <marker_namespace>sc_5_top</marker_namespace>
-      </plugin>
-    </sensor>
-  </gazebo>
-  <gazebo reference="grabbing_mechanism">
+        <marker_publish>sc_5_top</marker_publish>
+        <marker_id>9</marker_id>
+      </plugin>
+    </sensor>
     <sensor name='grabber_contact_sensor_sc_5_bot' type='contact'>
       <always_on>true</always_on>
       <update_rate>100</update_rate>
       <contact>
-        <collision>grabbing_mechanism_sc_5_bot_collision</collision>
+        <collision>grabbing_mechanism_sc_5_bot_collision_9</collision>
       </contact>
       <plugin name="contact_plugin_sc_5_bot" filename="libGrabberContactPlugin.so">
@@ -148,14 +139,13 @@
         <collision_y>-0.098</collision_y>
         <collision_z>-0.255</collision_z>
-        <marker_namespace>sc_5_bot</marker_namespace>
-      </plugin>
-    </sensor>
-  </gazebo>
-  <gazebo reference="grabbing_mechanism">
+        <marker_publish>sc_5_bot</marker_publish>
+        <marker_id>10</marker_id>
+      </plugin>
+    </sensor>
     <sensor name='grabber_contact_sensor_sc_6_top' type='contact'>
       <always_on>true</always_on>
       <update_rate>100</update_rate>
       <contact>
-        <collision>grabbing_mechanism_sc_6_top_collision</collision>
+        <collision>grabbing_mechanism_sc_6_top_collision_10</collision>
       </contact>
       <plugin name="contact_plugin_sc_6_top" filename="libGrabberContactPlugin.so">
@@ -163,14 +153,13 @@
         <collision_y>-0.098</collision_y>
         <collision_z>-0.135</collision_z>
-        <marker_namespace>sc_6_top</marker_namespace>
-      </plugin>
-    </sensor>
-  </gazebo>
-  <gazebo reference="grabbing_mechanism">
+        <marker_publish>sc_6_top</marker_publish>
+        <marker_id>11</marker_id>
+      </plugin>
+    </sensor>
     <sensor name='grabber_contact_sensor_sc_6_bot' type='contact'>
       <always_on>true</always_on>
       <update_rate>100</update_rate>
       <contact>
-        <collision>grabbing_mechanism_sc_6_bot_collision</collision>
+        <collision>grabbing_mechanism_sc_6_bot_collision_11</collision>
       </contact>
       <plugin name="contact_plugin_sc_6_bot" filename="libGrabberContactPlugin.so">
@@ -178,5 +167,6 @@
         <collision_y>-0.098</collision_y>
         <collision_z>-0.255</collision_z>
-        <marker_namespace>sc_6_bot</marker_namespace>
+        <marker_publish>sc_6_bot</marker_publish>
+        <marker_id>12</marker_id>
       </plugin>
     </sensor>
@@ -196,5 +186,5 @@
         </scan>
         <range>
-          <min>0.1</min>
+          <min>0.05</min>
           <max>30.0</max>
           <resolution>0.01</resolution>
@@ -222,5 +212,5 @@
         </scan>
         <range>
-          <min>0.1</min>
+          <min>0.05</min>
           <max>30.0</max>
           <resolution>0.01</resolution>
@@ -248,5 +238,5 @@
         </scan>
         <range>
-          <min>0.1</min>
+          <min>0.05</min>
           <max>30.0</max>
           <resolution>0.01</resolution>
@@ -274,5 +264,5 @@
         </scan>
         <range>
-          <min>0.1</min>
+          <min>0.05</min>
           <max>30.0</max>
           <resolution>0.01</resolution>
@@ -300,5 +290,5 @@
         </scan>
         <range>
-          <min>0.1</min>
+          <min>0.05</min>
           <max>30.0</max>
           <resolution>0.01</resolution>
@@ -326,5 +316,5 @@
         </scan>
         <range>
-          <min>0.1</min>
+          <min>0.05</min>
           <max>30.0</max>
           <resolution>0.01</resolution>

File: techtrix_description/urdf/techtrix.xacro (robot description, xacro)
@@ -103,4 +103,5 @@
   </joint>
   <link name="grabbing_mechanism">
+    <kinematic>true</kinematic>
     <collision name="grabbing_mechanism_sc_1_top">
       <origin xyz="0.551 -0.098 -0.135" rpy="${-pi/2} 0 0" />

Commit message: Add grabber command to pick up and drop

File: techtrix_description/urdf/gazebo_plugins.xacro (robot description, xacro)
@@ -5,5 +5,5 @@
     <sensor name='grabber_contact_sensor_sc_1_top' type='contact'>
       <always_on>true</always_on>
-      <update_rate>100</update_rate>
+      <update_rate>300</update_rate>
       <contact>
         <collision>grabbing_mechanism_sc_1_top_collision</collision>
@@ -19,5 +19,5 @@
     <sensor name='grabber_contact_sensor_sc_1_bot' type='contact'>
       <always_on>true</always_on>
-      <update_rate>100</update_rate>
+      <update_rate>300</update_rate>
       <contact>
         <collision>grabbing_mechanism_sc_1_bot_collision_1</collision>
@@ -33,5 +33,5 @@
     <sensor name='grabber_contact_sensor_sc_2_top' type='contact'>
       <always_on>true</always_on>
-      <update_rate>100</update_rate>
+      <update_rate>300</update_rate>
       <contact>
         <collision>grabbing_mechanism_sc_2_top_collision_2</collision>
@@ -47,5 +47,5 @@
     <sensor name='grabber_contact_sensor_sc_2_bot' type='contact'>
       <always_on>true</always_on>
-      <update_rate>100</update_rate>
+      <update_rate>300</update_rate>
       <contact>
         <collision>grabbing_mechanism_sc_2_bot_collision_3</collision>
@@ -61,5 +61,5 @@
     <sensor name='grabber_contact_sensor_sc_3_top' type='contact'>
       <always_on>true</always_on>
-      <update_rate>100</update_rate>
+      <update_rate>300</update_rate>
       <contact>
         <collision>grabbing_mechanism_sc_3_top_collision_4</collision>
@@ -75,5 +75,5 @@
     <sensor name='grabber_contact_sensor_sc_3_bot' type='contact'>
       <always_on>true</always_on>
-      <update_rate>100</update_rate>
+      <update_rate>300</update_rate>
       <contact>
         <collision>grabbing_mechanism_sc_3_bot_collision_5</collision>
@@ -89,5 +89,5 @@
     <sensor name='grabber_contact_sensor_sc_4_top' type='contact'>
       <always_on>true</always_on>
-      <update_rate>100</update_rate>
+      <update_rate>300</update_rate>
       <contact>
         <collision>grabbing_mechanism_sc_4_top_collision_6</collision>
@@ -103,5 +103,5 @@
     <sensor name='grabber_contact_sensor_sc_4_bot' type='contact'>
       <always_on>true</always_on>
-      <update_rate>100</update_rate>
+      <update_rate>300</update_rate>
       <contact>
         <collision>grabbing_mechanism_sc_4_bot_collision_7</collision>
@@ -117,5 +117,5 @@
     <sensor name='grabber_contact_sensor_sc_5_top' type='contact'>
       <always_on>true</always_on>
-      <update_rate>100</update_rate>
+      <update_rate>300</update_rate>
       <contact>
         <collision>grabbing_mechanism_sc_5_top_collision_8</collision>
@@ -131,5 +131,5 @@
     <sensor name='grabber_contact_sensor_sc_5_bot' type='contact'>
       <always_on>true</always_on>
-      <update_rate>100</update_rate>
+      <update_rate>300</update_rate>
       <contact>
         <collision>grabbing_mechanism_sc_5_bot_collision_9</collision>
@@ -145,5 +145,5 @@
     <sensor name='grabber_contact_sensor_sc_6_top' type='contact'>
       <always_on>true</always_on>
-      <update_rate>100</update_rate>
+      <update_rate>300</update_rate>
       <contact>
         <collision>grabbing_mechanism_sc_6_top_collision_10</collision>
@@ -159,5 +159,5 @@
     <sensor name='grabber_contact_sensor_sc_6_bot' type='contact'>
       <always_on>true</always_on>
-      <update_rate>100</update_rate>
+      <update_rate>300</update_rate>
       <contact>
         <collision>grabbing_mechanism_sc_6_bot_collision_11</collision>

File: techtrix_description/urdf/techtrix.xacro (robot description, xacro)
@@ -195,5 +195,5 @@
     <axis xyz="0 1 0" />
     <origin xyz="0 0 ${height/2}" />
-    <limit effort="1000.0" lower="0" upper="5.75" velocity="0.5" />
+    <limit effort="5000.0" lower="0" upper="5.75" velocity="0.5" />
   </joint>
   <joint name="lifting_joint" type="prismatic">
@@ -202,5 +202,5 @@
     <axis xyz="0 0 1" />
     <origin xyz="0 1.5 ${(height/2)-0.125}" />
-    <limit effort="1000.0" lower="-1.475" upper="0" velocity="0.25" />
+    <limit effort="6000.0" lower="-1.875" upper="0" velocity="0.25" />
     <dynamics damping="500" friction="20" />
   </joint>
@@ -209,5 +209,5 @@
     <child link="grabbing_mechanism" />
     <axis xyz="0 0 1" />
-    <limit effort="1000.0" lower="${-pi/2}" upper="0" velocity="0.5" />
+    <limit effort="5000.0" lower="${-pi/2}" upper="0" velocity="0.5" />
   </joint>
   <transmission name="base_transmission">
