Commit message: Attach robot to world/base_link

File: techtrix_description/urdf/techtrix.xacro (robot description, xacro)
@@ -10,9 +10,15 @@
   <xacro:property name="width" value="1" />
   <xacro:property name="height" value="1" />
-  <link name="base_link">
-    <xacro:default_inertial mass="1"/>
-  </link>
+  <!-- Used for fixing robot to Gazebo 'base_link' -->
+  <link name="world"/>
+  <joint name="base_joint" type="prismatic">
+    <parent link="world" />
+    <child link="chassis" />
+    <limit effort="1000.0" lower="-5" upper="0" velocity="0.5"/>
+    <axis xyz="0 1 0" />
+  </joint>
   <link name="chassis">
     <collision name="collision">
+      <origin xyz="0 0 ${height/2}" rpy="0 0 0" />
       <geometry>
         <box size="${width} ${length} ${height}" />
@@ -20,4 +26,5 @@
     </collision>
     <visual name="visual">
+      <origin xyz="0 0 ${height/2}" rpy="0 0 0" />
       <geometry>
         <box size="${width} ${length} ${height}" />
@@ -26,14 +33,4 @@
     <xacro:default_inertial mass="1"/>
   </link>
-  <joint name="base_joint" type="prismatic">
-    <parent link="base_link" />
-    <child link="chassis" />
-    <origin xyz="0 0 ${height/2}" />
-    <limit effort="1000.0" lower="-5" upper="0" velocity="0.5"/>
-    <axis xyz="0 1 0" />
-  </joint>
-  <gazebo reference="base_link">
-    <kinematic>true</kinematic>
-  </gazebo>
   <transmission name="base_transmission">
     <type>transmission_interface/SimpleTransmission</type>

Commit message: Remove unnecessary lines

File: techtrix_description/urdf/techtrix.xacro (robot description, xacro)
@@ -15,16 +15,15 @@
     <parent link="world" />
     <child link="chassis" />
+    <origin xyz="0 0 ${height/2}" />
     <limit effort="1000.0" lower="-5" upper="0" velocity="0.5"/>
     <axis xyz="0 1 0" />
   </joint>
   <link name="chassis">
-    <collision name="collision">
-      <origin xyz="0 0 ${height/2}" rpy="0 0 0" />
+    <collision>
       <geometry>
         <box size="${width} ${length} ${height}" />
       </geometry>
     </collision>
-    <visual name="visual">
-      <origin xyz="0 0 ${height/2}" rpy="0 0 0" />
+    <visual>
       <geometry>
         <box size="${width} ${length} ${height}" />

Commit message: Place robot in environment

File: techtrix_description/urdf/techtrix.xacro (robot description, xacro)
@@ -7,7 +7,7 @@
     </inertial>
   </xacro:macro>
-  <xacro:property name="length" value="1" />
+  <xacro:property name="length" value="1.5" />
   <xacro:property name="width" value="1" />
-  <xacro:property name="height" value="1" />
+  <xacro:property name="height" value="2.5" />
   <!-- Used for fixing robot to Gazebo 'base_link' -->
   <link name="world"/>
@@ -16,5 +16,5 @@
     <child link="chassis" />
     <origin xyz="0 0 ${height/2}" />
-    <limit effort="1000.0" lower="-5" upper="0" velocity="0.5"/>
+    <limit effort="1000.0" lower="0" upper="6.5" velocity="0.5"/>
     <axis xyz="0 1 0" />
   </joint>

Commit message: Apply mesh on robot

File: techtrix_description/urdf/techtrix.xacro (robot description, xacro)
@@ -7,7 +7,8 @@
     </inertial>
   </xacro:macro>
-  <xacro:property name="length" value="1.5" />
-  <xacro:property name="width" value="1" />
-  <xacro:property name="height" value="2.5" />
+  <xacro:property name="pi" value="3.1415926535897931" />
+  <xacro:property name="length" value="1.6" />
+  <xacro:property name="width" value="1.5" />
+  <xacro:property name="height" value="2.3" />
   <!-- Used for fixing robot to Gazebo 'base_link' -->
   <link name="world"/>
@@ -16,5 +17,5 @@
     <child link="chassis" />
     <origin xyz="0 0 ${height/2}" />
-    <limit effort="1000.0" lower="0" upper="6.5" velocity="0.5"/>
+    <limit effort="1000.0" lower="0" upper="5.75" velocity="0.5" />
     <axis xyz="0 1 0" />
   </joint>
@@ -26,6 +27,7 @@
     </collision>
     <visual>
+      <origin xyz="0 0.375 -2.355" rpy="0 0 ${-pi/2}" />
       <geometry>
-        <box size="${width} ${length} ${height}" />
+        <mesh filename="package://techtrix_description/meshes/techtrix_frame.dae" scale="${1/3} ${1/3} ${1/3}" />
       </geometry>
     </visual>

Commit message: Move robot into place and disable collisions

File: techtrix_description/urdf/techtrix.xacro (robot description, xacro)
@@ -21,9 +21,9 @@
   </joint>
   <link name="chassis">
-    <collision>
+    <!-- <collision>
       <geometry>
         <box size="${width} ${length} ${height}" />
       </geometry>
-    </collision>
+    </collision> -->
     <visual>
       <origin xyz="0 0.375 -2.355" rpy="0 0 ${-pi/2}" />

Commit message: Add grabber

File: techtrix_description/urdf/techtrix.xacro (robot description, xacro)
@@ -34,4 +34,26 @@
     <xacro:default_inertial mass="1"/>
   </link>
+  <link name="grabber">
+    <!-- <collision>
+      <origin xyz="0 0 -0.015" />
+      <geometry>
+        <box size="1.375 0.26 0.03" />
+      </geometry>
+    </collision> -->
+    <visual>
+      <origin xyz="0 -1.133 -2.7575" rpy="0 0 ${-pi/2}" />
+      <geometry>
+        <mesh filename="package://techtrix_description/meshes/techtrix_grabber.dae" scale="${1/3} ${1/3} ${1/3}" />
+      </geometry>
+    </visual>
+    <xacro:default_inertial mass="1"/>
+  </link>
+  <joint name="lifting_joint" type="prismatic">
+    <parent link="chassis" />
+    <child link="grabber" />
+    <origin xyz="0 1.5 ${(height/2)-0.075}" />
+    <limit effort="1000.0" lower="0" upper="-1.5" velocity=".1" />
+    <axis xyz="0 0 1" />
+  </joint>
   <transmission name="base_transmission">
     <type>transmission_interface/SimpleTransmission</type>

Commit message: Implement bearing

File: techtrix_description/urdf/techtrix.xacro (robot description, xacro)
@@ -13,12 +13,5 @@
   <!-- Used for fixing robot to Gazebo 'base_link' -->
   <link name="world"/>
-  <joint name="base_joint" type="prismatic">
-    <parent link="world" />
-    <child link="chassis" />
-    <origin xyz="0 0 ${height/2}" />
-    <limit effort="1000.0" lower="0" upper="5.75" velocity="0.5" />
-    <axis xyz="0 1 0" />
-  </joint>
-  <link name="chassis">
+  <link name="frame">
     <!-- <collision>
       <geometry>
@@ -34,11 +27,14 @@
     <xacro:default_inertial mass="1"/>
   </link>
+  <link name="bearing">
+    <xacro:default_inertial mass="1"/>
+  </link>
   <link name="grabber">
-    <!-- <collision>
+    <collision>
       <origin xyz="0 0 -0.015" />
       <geometry>
         <box size="1.375 0.26 0.03" />
       </geometry>
-    </collision> -->
+    </collision>
     <visual>
       <origin xyz="0 -1.133 -2.7575" rpy="0 0 ${-pi/2}" />
@@ -49,10 +45,23 @@
     <xacro:default_inertial mass="1"/>
   </link>
+  <joint name="base_joint" type="prismatic">
+    <parent link="world" />
+    <child link="frame" />
+    <axis xyz="0 1 0" />
+    <origin xyz="0 0 ${height/2}" />
+    <limit effort="1000.0" lower="0" upper="5.75" velocity="0.5" />
+  </joint>
   <joint name="lifting_joint" type="prismatic">
-    <parent link="chassis" />
+    <parent link="frame" />
+    <child link="bearing" />
+    <axis xyz="0 0 1" />
+    <origin xyz="0 1.5 ${(height/2)-0.125}" />
+    <limit effort="1000.0" lower="-1.475" upper="0" velocity="0.1" />
+  </joint>
+  <joint name="rotating_joint" type="revolute">
+    <parent link="bearing" />
     <child link="grabber" />
-    <origin xyz="0 1.5 ${(height/2)-0.075}" />
-    <limit effort="1000.0" lower="0" upper="-1.5" velocity=".1" />
     <axis xyz="0 0 1" />
+    <limit effort="1000.0" lower="${-pi/2}" upper="0" velocity="0.5" />
   </joint>
   <transmission name="base_transmission">

Commit message: Implement motors for lifting and rotating

File: techtrix_description/urdf/techtrix.xacro (robot description, xacro)
@@ -75,4 +75,24 @@
     </actuator>
   </transmission>
+  <transmission name="lifting_transmission">
+    <type>transmission_interface/SimpleTransmission</type>
+    <joint name="lifting_joint">
+      <hardwareInterface>hardware_interface/EffortJointInterface</hardwareInterface>
+    </joint>
+    <actuator name="lifting_motor">
+      <hardwareInterface>hardware_interface/EffortJointInterface</hardwareInterface>
+      <mechanicalReduction>1</mechanicalReduction>
+    </actuator>
+  </transmission>
+  <transmission name="rotating_transmission">
+    <type>transmission_interface/SimpleTransmission</type>
+    <joint name="rotating_joint">
+      <hardwareInterface>hardware_interface/EffortJointInterface</hardwareInterface>
+    </joint>
+    <actuator name="rotating_motor">
+      <hardwareInterface>hardware_interface/EffortJointInterface</hardwareInterface>
+      <mechanicalReduction>1</mechanicalReduction>
+    </actuator>
+  </transmission>
   <gazebo>
     <plugin name="gazebo_ros_control" filename="libgazebo_ros_control.so">

Commit message: Fix joint behaviour

File: techtrix_description/urdf/techtrix.xacro (robot description, xacro)
@@ -57,5 +57,6 @@
     <axis xyz="0 0 1" />
     <origin xyz="0 1.5 ${(height/2)-0.125}" />
-    <limit effort="1000.0" lower="-1.475" upper="0" velocity="0.1" />
+    <limit effort="1000.0" lower="-1.475" upper="0" velocity="0.25" />
+    <dynamics damping="500" friction="20" />
   </joint>
   <joint name="rotating_joint" type="revolute">

Commit message: Rename grabber

File: techtrix_description/urdf/techtrix.xacro (robot description, xacro)
@@ -30,5 +30,5 @@
     <xacro:default_inertial mass="1"/>
   </link>
-  <link name="grabber">
+  <link name="grabbing_mechanism">
     <collision>
       <origin xyz="0 0 -0.015" />
@@ -40,5 +40,5 @@
       <origin xyz="0 -1.133 -2.7575" rpy="0 0 ${-pi/2}" />
       <geometry>
-        <mesh filename="package://techtrix_description/meshes/techtrix_grabber.dae" scale="${1/3} ${1/3} ${1/3}" />
+        <mesh filename="package://techtrix_description/meshes/techtrix_grabbing_mechanism.dae" scale="${1/3} ${1/3} ${1/3}" />
       </geometry>
     </visual>
@@ -62,5 +62,5 @@
   <joint name="rotating_joint" type="revolute">
     <parent link="bearing" />
-    <child link="grabber" />
+    <child link="grabbing_mechanism" />
     <axis xyz="0 0 1" />
     <limit effort="1000.0" lower="${-pi/2}" upper="0" velocity="0.5" />

Commit message: Updated robot to include the thermal sensor

File: techtrix_description/urdf/techtrix.xacro (robot description, xacro)
@@ -1,14 +1,8 @@
 <?xml version="1.0"?>
 <robot xmlns:xacro="http://www.ros.org/wiki/xacro" name="techtrix_robot">
-  <xacro:macro name="default_inertial" params="mass">
-    <inertial>
-      <mass value="${mass}" />
-      <inertia ixx="1.0" ixy="0.0" ixz="0.0" iyy="1.0" iyz="0.0" izz="1.0" />
-    </inertial>
-  </xacro:macro>
-  <xacro:property name="pi" value="3.1415926535897931" />
-  <xacro:property name="length" value="1.6" />
-  <xacro:property name="width" value="1.5" />
-  <xacro:property name="height" value="2.3" />
+  <xacro:include filename="$(find techtrix_description)/urdf/macros.xacro"/>
+  <xacro:include filename="$(find techtrix_description)/urdf/techtrix_properties.xacro"/>
+  <xacro:include filename="$(find techtrix_description)/urdf/materials.xacro"/>
+  <xacro:include filename="$(find techtrix_description)/urdf/gazebo_plugins.xacro"/>
   <!-- Used for fixing robot to Gazebo 'base_link' -->
   <link name="world"/>
@@ -45,4 +39,25 @@
     <xacro:default_inertial mass="1"/>
   </link>
+  <!-- Camera -->
+  <link name="camera_link">
+    <collision>
+      <origin xyz="0 0 0" rpy="0 0 0"/>
+      <geometry>
+	      <box size="${camera_link} ${camera_link} ${camera_link}"/>
+      </geometry>
+    </collision>
+    <visual>
+      <origin xyz="0 0 0" rpy="0 0 0"/>
+      <geometry>
+	      <box size="${camera_link} ${camera_link} ${camera_link}"/>
+      </geometry>
+      <material name="red"/>
+    </visual>
+    <inertial>
+      <mass value="1e-5" />
+      <origin xyz="0 0 0" rpy="0 0 0"/>
+      <inertia ixx="1e-6" ixy="0" ixz="0" iyy="1e-6" iyz="0" izz="1e-6" />
+    </inertial>
+  </link>
   <joint name="base_joint" type="prismatic">
     <parent link="world" />
@@ -64,4 +79,10 @@
     <axis xyz="0 0 1" />
     <limit effort="1000.0" lower="${-pi/2}" upper="0" velocity="0.5" />
+  </joint>
+  <joint name="camera_joint" type="fixed">
+    <parent link="frame"/>
+    <child link="camera_link"/>
+    <axis xyz="0 1 0" />
+    <origin xyz="${camera_link} 0 1" rpy="0 0 0"/>
   </joint>
   <transmission name="base_transmission">

Commit message: Create collision box for frame

File: techtrix_description/urdf/techtrix.xacro (robot description, xacro)
@@ -8,9 +8,34 @@
   <link name="world"/>
   <link name="frame">
-    <!-- <collision>
+    <collision>
+      <origin xyz="0 0 ${(-height/2)+0.19}" />
       <geometry>
-        <box size="${width} ${length} ${height}" />
+        <box size="${width} ${length} 0.3" />
       </geometry>
-    </collision> -->
+    </collision>
+    <collision>
+      <origin xyz="0 0 ${(height/2)-0.045}" />
+      <geometry>
+        <box size="${width} ${length} 0.12" />
+      </geometry>
+    </collision>
+    <collision>
+      <origin xyz="0 0.745 ${(height/2)-0.045}" />
+      <geometry>
+        <box size="${width} ${length} 0.12" />
+      </geometry>
+    </collision>
+    <collision>
+      <origin xyz="${(width/2)-0.03} 0 0" />
+      <geometry>
+        <box size="0.1 ${length} ${height}" />
+      </geometry>
+    </collision>
+    <collision>
+      <origin xyz="${(-width/2)+0.03} 0 0" />
+      <geometry>
+        <box size="0.1 ${length} ${height}" />
+      </geometry>
+    </collision>
     <visual>
       <origin xyz="0 0.375 -2.355" rpy="0 0 ${-pi/2}" />
@@ -44,5 +69,5 @@
       <origin xyz="0 0 0" rpy="0 0 0"/>
       <geometry>
-	      <box size="${camera_link} ${camera_link} ${camera_link}"/>
+        <box size="${camera_link} ${camera_link} ${camera_link}"/>
       </geometry>
     </collision>
@@ -50,5 +75,5 @@
       <origin xyz="0 0 0" rpy="0 0 0"/>
       <geometry>
-	      <box size="${camera_link} ${camera_link} ${camera_link}"/>
+        <box size="${camera_link} ${camera_link} ${camera_link}"/>
       </geometry>
       <material name="yellow">

Commit message: Fixed camera angle

File: techtrix_description/urdf/techtrix.xacro (robot description, xacro)
@@ -52,7 +52,4 @@
 	      <box size="${camera_link} ${camera_link} ${camera_link}"/>
       </geometry>
-      <material name="yellow">
-        <color rgba="1 1 0 1"/>
-      </material>
     </visual>
     <inertial>
@@ -86,5 +83,5 @@
     <child link="camera_link"/>
     <axis xyz="0 1 0" />
-    <origin xyz="${camera_link} 0 1" rpy="0 0 0"/>
+    <origin xyz="${camera_link} 0 1" rpy="0 0 -1.6"/>
   </joint>
   <transmission name="base_transmission">

Commit message: Add contact sensors

File: techtrix_description/urdf/techtrix.xacro (robot description, xacro)
@@ -1,14 +1,8 @@
 <?xml version="1.0"?>
 <robot xmlns:xacro="http://www.ros.org/wiki/xacro" name="techtrix_robot">
-  <xacro:macro name="default_inertial" params="mass">
-    <inertial>
-      <mass value="${mass}" />
-      <inertia ixx="1.0" ixy="0.0" ixz="0.0" iyy="1.0" iyz="0.0" izz="1.0" />
-    </inertial>
-  </xacro:macro>
-  <xacro:property name="pi" value="3.1415926535897931" />
-  <xacro:property name="length" value="1.6" />
-  <xacro:property name="width" value="1.5" />
-  <xacro:property name="height" value="2.3" />
+  <xacro:include filename="$(find techtrix_description)/urdf/macros.xacro"/>
+  <xacro:include filename="$(find techtrix_description)/urdf/techtrix_properties.xacro"/>
+  <xacro:include filename="$(find techtrix_description)/urdf/materials.xacro"/>
+  <xacro:include filename="$(find techtrix_description)/urdf/gazebo_plugins.xacro"/>
   <!-- Used for fixing robot to Gazebo 'base_link' -->
   <link name="world"/>
@@ -31,5 +25,77 @@
   </link>
   <link name="grabbing_mechanism">
-    <collision>
+    <collision name="grabbing_mechanism_sc_1_top">
+      <origin xyz="0.551 -0.098 -0.135" rpy="${-pi/2} 0 0" />
+      <geometry>
+        <cylinder radius="0.03" length="0.001" turns="0.5"/>
+      </geometry>
+    </collision>
+    <collision name="grabbing_mechanism_sc_1_bot">
+      <origin xyz="0.551 -0.098 -0.255" rpy="${-pi/2} 0 0" />
+      <geometry>
+        <cylinder radius="0.03" length="0.001" turns="0.5"/>
+      </geometry>
+    </collision>
+    <collision name="grabbing_mechanism_sc_2_top">
+      <origin xyz="0.339 -0.098 -0.135" rpy="${-pi/2} 0 0" />
+      <geometry>
+        <cylinder radius="0.03" length="0.001" turns="0.5"/>
+      </geometry>
+    </collision>
+    <collision name="grabbing_mechanism_sc_2_bot">
+      <origin xyz="0.339 -0.098 -0.255" rpy="${-pi/2} 0 0" />
+      <geometry>
+        <cylinder radius="0.03" length="0.001" turns="0.5"/>
+      </geometry>
+    </collision>
+    <collision name="grabbing_mechanism_sc_3_top">
+      <origin xyz="0.127 -0.098 -0.135" rpy="${-pi/2} 0 0" />
+      <geometry>
+        <cylinder radius="0.03" length="0.001" turns="0.5"/>
+      </geometry>
+    </collision>
+    <collision name="grabbing_mechanism_sc_3_bot">
+      <origin xyz="0.127 -0.098 -0.255" rpy="${-pi/2} 0 0" />
+      <geometry>
+        <cylinder radius="0.03" length="0.001" turns="0.5"/>
+      </geometry>
+    </collision>
+    <collision name="grabbing_mechanism_sc_4_top">
+      <origin xyz="-0.127 -0.098 -0.135" rpy="${-pi/2} 0 0" />
+      <geometry>
+        <cylinder radius="0.03" length="0.001" turns="0.5"/>
+      </geometry>
+    </collision>
+    <collision name="grabbing_mechanism_sc_4_bot">
+      <origin xyz="-0.127 -0.098 -0.255" rpy="${-pi/2} 0 0" />
+      <geometry>
+        <cylinder radius="0.03" length="0.001" turns="0.5"/>
+      </geometry>
+    </collision>
+    <collision name="grabbing_mechanism_sc_5_top">
+      <origin xyz="-0.339 -0.098 -0.135" rpy="${-pi/2} 0 0" />
+      <geometry>
+        <cylinder radius="0.03" length="0.001" turns="0.5"/>
+      </geometry>
+    </collision>
+    <collision name="grabbing_mechanism_sc_5_bot">
+      <origin xyz="-0.339 -0.098 -0.255" rpy="${-pi/2} 0 0" />
+      <geometry>
+        <cylinder radius="0.03" length="0.001" turns="0.5"/>
+      </geometry>
+    </collision>
+    <collision name="grabbing_mechanism_sc_6_top">
+      <origin xyz="-0.551 -0.098 -0.135" rpy="${-pi/2} 0 0" />
+      <geometry>
+        <cylinder radius="0.03" length="0.001" turns="0.5"/>
+      </geometry>
+    </collision>
+    <collision name="grabbing_mechanism_sc_6_bot">
+      <origin xyz="-0.551 -0.098 -0.255" rpy="${-pi/2} 0 0" />
+      <geometry>
+        <cylinder radius="0.03" length="0.001" turns="0.5"/>
+      </geometry>
+    </collision>
+    <collision name="grabbing_mechanism_top">
       <origin xyz="0 0 -0.015" />
       <geometry>

Commit message: Finished implementation of robot movement

File: techtrix_description/urdf/techtrix.xacro (robot description, xacro)
@@ -231,5 +231,5 @@
     <axis xyz="0 1 0" />
     <origin xyz="0 0 ${height/2}" />
-    <limit effort="5000.0" lower="0" upper="5.75" velocity="0.5" />
+    <limit effort="10000.0" lower="0" upper="5.75" velocity="1" />
   </joint>
   <joint name="lifting_joint" type="prismatic">
@@ -238,5 +238,5 @@
     <axis xyz="0 0 1" />
     <origin xyz="0 1.5 ${(height/2)-0.125}" />
-    <limit effort="6000.0" lower="-1.875" upper="0" velocity="0.25" />
+    <limit effort="10000.0" lower="-1.875" upper="0" velocity="0.25" />
     <dynamics damping="500" friction="20" />
   </joint>
